Commit message: chenges

File: uuv_sensor_plugins/uuv_sensor_ros_plugins/urdf/camera_snippets.xacro (robot description, xacro)
@@ -122,4 +122,5 @@
         </camera>
         <plugin name="camera${suffix}_controller" filename="libgazebo_ros_camera.so">
+          <!-- <alwaysOn>true</alwaysOn> -->
           <updateRate>${update_rate}</updateRate>
           <cameraName>${namespace}/camera${suffix}</cameraName>

File: uuv_sensor_plugins/uuv_sensor_ros_plugins/urdf/sensor_snippets.xacro (robot description, xacro)
@@ -24,3 +24,7 @@
   <xacro:include filename="$(find uuv_sensor_ros_plugins)/urdf/pose_3d_snippets.xacro" />
   <xacro:include filename="$(find uuv_sensor_ros_plugins)/urdf/chemical_concentration_snippets.xacro"/>
+  <xacro:include filename="$(find uuv_sensor_ros_plugins)/urdf/sonar_sensor.urdf.xacro"/>
+<!--  <xacro:include filename="$(find uuv_sensor_ros_plugins)/urdf/kinect_v2.urdf.xacro"/>-->
+  <xacro:include filename="$(find uuv_sensor_ros_plugins)/urdf/camera.urdf.xacro"/>
+<!--  <xacro:include filename="$(find uuv_sensor_ros_plugins)/urdf/kinect.urdf.xacro"/>-->
 </robot>

File: uuv_sensor_plugins/uuv_sensor_ros_plugins/urdf/sonar_sensor.urdf.xacro (robot description, xacro)
@@ -1,8 +1,8 @@
 <?xml version="1.0"?>
 <robot xmlns:xacro="http://ros.org/wiki/xacro">
-  <xacro:macro name="sonar_sensor" params="name parent *origin ros_topic update_rate min_range max_range field_of_view ray_count">
+  <xacro:macro name="sonar_sensor" params="name parent_link *origin ros_topic update_rate min_range max_range field_of_view ray_count">
     <joint name="${name}_joint" type="fixed">
       <xacro:insert_block name="origin" />
-      <parent link="${parent}"/>
+      <parent link="${parent_link}"/>
       <child link="${name}_link"/>
     </joint>
@@ -17,5 +17,5 @@
         <geometry>
           <!--<box size="0.01 0.01 0.01" /> -->
-          <mesh filename="package://hector_sensors_description/meshes/sonar_sensor/max_sonar_ez4.dae"/>
+          <mesh filename="file://$(find uuv_sensor_ros_plugins)/meshes/sonar_sensor/max_sonar_ez4.dae"/>
         </geometry>
       </visual>
